File: kevins-pcb-numpad/_autosave-kevins-pcb-numpad.kicad_pcb (KiCad board)
At the start: 2 copper layers, 24 parts, among them SW1 SW_Push, U1 ATmega32U4-AU, Y1 16MHz

Commit message: Final
Routing:
- net COL1: track 55.4 -> 19.0 mm
- added copper zone on B.Cu, net GND
Changed lines of the file:
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@@
     (thickness 1.6)
     (drawings 9)
-    (tracks 189)
+    (tracks 187)
     (zones 0)
     (modules 24)
@@
     (visible_elements FFFFFF7F)
     (pcbplotparams
-      (layerselection 0x010fc_ffffffff)
-      (usegerberextensions false)
+      (layerselection 0x010f0_ffffffff)
+      (usegerberextensions true)
       (usegerberattributes true)
       (usegerberadvancedattributes true)
-      (creategerberjobfile true)
+      (creategerberjobfile false)
       (excludeedgelayer true)
       (linewidth 0.100000)
@@
       (plotinvisibletext false)
       (padsonsilk false)
-      (subtractmaskfromsilk false)
+      (subtractmaskfromsilk true)
       (outputformat 1)
       (mirror false)
-      (drillshape 1)
+      (drillshape 0)
       (scaleselection 1)
-      (outputdirectory ""))
+      (outputdirectory "../../../../3D Objects/Gerbers/"))
   )
   (net 0 "")
@@
     (fp_line (start 1.68 0.95) (end 1.68 -0.95) (layer B.CrtYd) (width 0.05))
     (fp_line (start 1.68 -0.95) (end -1.68 -0.95) (layer B.CrtYd) (width 0.05))
-    (pad 2 smd roundrect (at 0.9125 0 90) (size 1.025 1.4) (layers B.Cu B.Paste B.Mask) (roundrect_rratio 0.243902)
+    (pad 2 smd roundrect (at 0.9125 0 90) (size 1.025 1.4) (layers B.Cu B.Paste B.Mask) (roundrect_rratio 0.2439014634146341)
       (net 20 "Net-(R4-Pad2)"))
-    (pad 1 smd roundrect (at -0.9125 0 90) (size 1.025 1.4) (layers B.Cu B.Paste B.Mask) (roundrect_rratio 0.243902)
+    (pad 1 smd roundrect (at -0.9125 0 90) (size 1.025 1.4) (layers B.Cu B.Paste B.Mask) (roundrect_rratio 0.2439014634146341)
       (net 1 GND))
     (model ${KISYS3DMOD}/Resistor_SMD.3dshapes/R_0805_2012Metric.wrl
@@
       (effects (font (size 0.5 0.5) (thickness 0.08)) (justify mirror))
     )
-    (pad 1 smd roundrect (at -0.9125 0 270) (size 1.025 1.4) (layers B.Cu B.Paste B.Mask) (roundrect_rratio 0.243902)
+    (pad 1 smd roundrect (at -0.9125 0 270) (size 1.025 1.4) (layers B.Cu B.Paste B.Mask) (roundrect_rratio 0.2439014634146341)
       (net 2 +5V))
-    (pad 2 smd roundrect (at 0.9125 0 270) (size 1.025 1.4) (layers B.Cu B.Paste B.Mask) (roundrect_rratio 0.243902)
+    (pad 2 smd roundrect (at 0.9125 0 270) (size 1.025 1.4) (layers B.Cu B.Paste B.Mask) (roundrect_rratio 0.2439014634146341)
       (net 19 "Net-(R3-Pad2)"))
     (model ${KISYS3DMOD}/Resistor_SMD.3dshapes/R_0805_2012Metric.wrl
@@
     (fp_line (start 1.68 0.95) (end 1.68 -0.95) (layer B.CrtYd) (width 0.05))
     (fp_line (start 1.68 -0.95) (end -1.68 -0.95) (layer B.CrtYd) (width 0.05))
-    (pad 2 smd roundrect (at 0.9125 0 90) (size 1.025 1.4) (layers B.Cu B.Paste B.Mask) (roundrect_rratio 0.243902)
+    (pad 2 smd roundrect (at 0.9125 0 90) (size 1.025 1.4) (layers B.Cu B.Paste B.Mask) (roundrect_rratio 0.2439014634146341)
       (net 17 D+))
-    (pad 1 smd roundrect (at -0.9125 0 90) (size 1.025 1.4) (layers B.Cu B.Paste B.Mask) (roundrect_rratio 0.243902)
+    (pad 1 smd roundrect (at -0.9125 0 90) (size 1.025 1.4) (layers B.Cu B.Paste B.Mask) (roundrect_rratio 0.2439014634146341)
       (net 18 "Net-(R2-Pad1)"))
     (model ${KISYS3DMOD}/Resistor_SMD.3dshapes/R_0805_2012Metric.wrl
@@
     (fp_line (start 1.68 0.95) (end 1.68 -0.95) (layer B.CrtYd) (width 0.05))
     (fp_line (start 1.68 -0.95) (end -1.68 -0.95) (layer B.CrtYd) (width 0.05))
-    (pad 2 smd roundrect (at 0.9125 0 90) (size 1.025 1.4) (layers B.Cu B.Paste B.Mask) (roundrect_rratio 0.243902)
+    (pad 2 smd roundrect (at 0.9125 0 90) (size 1.025 1.4) (layers B.Cu B.Paste B.Mask) (roundrect_rratio 0.2439014634146341)
       (net 15 D-))
-    (pad 1 smd roundrect (at -0.9125 0 90) (size 1.025 1.4) (layers B.Cu B.Paste B.Mask) (roundrect_rratio 0.243902)
+    (pad 1 smd roundrect (at -0.9125 0 90) (size 1.025 1.4) (layers B.Cu B.Paste B.Mask) (roundrect_rratio 0.2439014634146341)
       (net 16 "Net-(R1-Pad1)"))
     (model ${KISYS3DMOD}/Resistor_SMD.3dshapes/R_0805_2012Metric.wrl
@@
   (segment (start 61.697 104.41075) (end 61.697 101.082848) (width 0.381) (layer B.Cu) (net 1))
   (segment (start 55.99299 88.75899) (end 56.896 89.662) (width 0.381) (layer B.Cu) (net 1))
-  (segment (start 45.25625 86.460596) (end 47.554644 88.75899) (width 0.381) (layer B.Cu) (net 1))
-  (segment (start 45.25625 86.25625) (end 45.25625 86.460596) (width 0.381) (layer B.Cu) (net 1))
   (segment (start 63.297 94.14175) (end 64.91325 95.758) (width 0.381) (layer B.Cu) (net 1))
   (segment (start 63.297 93.01075) (end 63.297 94.14175) (width 0.381) (layer B.Cu) (net 1))
@@
   (segment (start 49.54401 88.75899) (end 55.99299 88.75899) (width 0.381) (layer B.Cu) (net 1))
   (segment (start 47.554644 88.75899) (end 49.54401 88.75899) (width 0.381) (layer B.Cu) (net 1))
+  (segment (start 45.25625 86.25625) (end 45.25625 86.460596) (width 0.381) (layer B.Cu) (net 1))
+  (segment (start 45.25625 86.460596) (end 47.554644 88.75899) (width 0.381) (layer B.Cu) (net 1))
   (segment (start 74.05275 95.51075) (end 70.597 95.51075) (width 0.381) (layer B.Cu) (net 2))
   (segment (start 74.676 96.134) (end 74.05275 95.51075) (width 0.381) (layer B.Cu) (net 2))
@@
   (segment (start 113.792 106.172) (end 110.49 102.87) (width 0.254) (layer B.Cu) (net 11))
   (segment (start 115.443 106.172) (end 113.792 106.172) (width 0.254) (layer B.Cu) (net 11))
-  (segment (start 42.05625 86.370793) (end 42.05625 86.25625) (width 0.254) (layer B.Cu) (net 12))
   (segment (start 38.735 89.692043) (end 40.289043 88.138) (width 0.254) (layer B.Cu) (net 12))
   (segment (start 38.735 93.472) (end 38.735 89.692043) (width 0.254) (layer B.Cu) (net 12))
+  (segment (start 40.289043 88.138) (end 41.529 88.138) (width 0.254) (layer B.Cu) (net 12))
+  (segment (start 42.05625 86.370793) (end 42.05625 86.25625) (width 0.254) (layer B.Cu) (net 12))
+  (segment (start 41.529 88.138) (end 42.05625 87.61075) (width 0.254) (layer B.Cu) (net 12))
   (segment (start 42.05625 87.61075) (end 42.05625 86.25625) (width 0.254) (layer B.Cu) (net 12))
-  (segment (start 41.529 88.138) (end 42.05625 87.61075) (width 0.254) (layer B.Cu) (net 12))
-  (segment (start 40.289043 88.138) (end 41.529 88.138) (width 0.254) (layer B.Cu) (net 12))
   (segment (start 81.96075 99.51075) (end 86.4 103.95) (width 0.254) (layer B.Cu) (net 13))
   (segment (start 70.597 99.51075) (end 81.96075 99.51075) (width 0.254) (layer B.Cu) (net 13))
@@
   (segment (start 86.4 103.95) (end 86.106 103.656) (width 0.254) (layer F.Cu) (net 13))
   (segment (start 104.14 86.36) (end 104.14 105.41) (width 0.254) (layer F.Cu) (net 14))
-  (segment (start 97.44075 98.71075) (end 70.597 98.71075) (width 0.254) (layer B.Cu) (net 14))
-  (segment (start 104.14 105.41) (end 97.44075 98.71075) (width 0.254) (layer B.Cu) (net 14))
   (segment (start 41.529 90.932) (end 41.529 90.805) (width 0.254) (layer B.Cu) (net 15))
+  (segment (start 41.529 90.932) (end 42.85625 89.60475) (width 0.254) (layer B.Cu) (net 15))
   (segment (start 42.926 86.326) (end 42.85625 86.25625) (width 0.254) (layer B.Cu) (net 15))
   (segment (start 42.85625 89.60475) (end 42.85625 86.25625) (width 0.254) (layer B.Cu) (net 15))
-  (segment (start 41.529 90.932) (end 42.85625 89.60475) (width 0.254) (layer B.Cu) (net 15))
   (segment (start 59.17825 101.092) (end 59.197 101.11075) (width 0.254) (layer B.Cu) (net 16))
   (segment (start 42.85299 101.01899) (end 42.926 101.092) (width 0.254) (layer B.Cu) (net 16))
@@
   (segment (start 42.85299 95.04999) (end 42.85299 101.01899) (width 0.254) (layer B.Cu) (net 16))
   (segment (start 42.926 101.092) (end 59.17825 101.092) (width 0.254) (layer B.Cu) (net 16))
+  (segment (start 44.704 90.932) (end 43.65625 89.88425) (width 0.254) (layer B.Cu) (net 17))
   (segment (start 44.704 90.932) (end 44.704 90.424) (width 0.254) (layer B.Cu) (net 17))
   (segment (start 43.688 86.288) (end 43.65625 86.25625) (width 0.254) (layer B.Cu) (net 17))
   (segment (start 43.65625 89.88425) (end 43.65625 86.25625) (width 0.254) (layer B.Cu) (net 17))
-  (segment (start 44.704 90.932) (end 43.65625 89.88425) (width 0.254) (layer B.Cu) (net 17))
   (segment (start 59.17775 100.33) (end 59.197 100.31075) (width 0.254) (layer B.Cu) (net 18))
   (segment (start 43.307 100.33) (end 59.17775 100.33) (width 0.254) (layer B.Cu) (net 18))
@@
   (segment (start 70.69175 102.616) (end 70.597 102.71075) (width 0.254) (layer B.Cu) (net 20))
   (segment (start 74.549 102.616) (end 70.69175 102.616) (width 0.254) (layer B.Cu) (net 20))
+  (zone (net 1) (net_name GND) (layer B.Cu) (hatch edge 0.508)
+    (connect_pads (clearance 0.508))
+    (min_thickness 0.254)
+    (fill yes (arc_segments 32) (thermal_gap 0.508) (thermal_bridge_width 0.508))
+    (polygon
+      (pts
+        (xy 73.66 91.948) (xy 56.769 92.075) (xy 56.769 82.804) (xy 73.66 82.804)
+      )
+    )
+  )
+  (zone (net 1) (net_name GND) (layer B.Cu) (hatch edge 0.508)
+    (connect_pads (clearance 0.508))
+    (min_thickness 0.254)
+    (fill yes (arc_segments 32) (thermal_gap 0.508) (thermal_bridge_width 0.508))
+    (polygon
+      (pts
+        (xy 69.469 103.251) (xy 60.198 103.251) (xy 60.198 94.107) (xy 69.596 94.107)
+      )
+    )
+  )
+  (zone (net 1) (net_name GND) (layer B.Cu) (hatch edge 0.508)
+    (connect_pads (clearance 0.508))
+    (min_thickness 0.254)
+    (fill yes (arc_segments 32) (thermal_gap 0.508) (thermal_bridge_width 0.508))
+    (polygon
+      (pts
+        (xy 47.371 87.63) (xy 39.751 87.249) (xy 39.751 80.391) (xy 47.371 80.391)
+      )
+    )
+  )
 )
